File: Hardware/G2G-U Module/G2G-U Module.brd (EAGLE design)
At the start: 13.1 x 12.8 mm, 3 parts, among them J1 GROVE-4P-2.0-3470130P1

Commit message: Added frames to the U and X module schematics.
Parts:
- added FRAME1: (no value), SparkFun-Aesthetics:DUMMY
Changed lines of the file:
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@@
 <element name="LOGO1" library="SparkFun-Aesthetics" package="OSHW-LOGO-S" value="OSHW-LOGOS" x="1.8796" y="1.778" rot="MR0"/>
 <element name="U$1" library="SoftDust" package="2X5_1.27MM_FEMALE_PLUG" value="2X5_1.27MM_FEMALE_PLUG" x="6.5532" y="9.9822" rot="MR0"/>
+<element name="FRAME1" library="SparkFun-Aesthetics" package="DUMMY" value="" x="0" y="-1.27">
+<attribute name="VERSION" value="v1.0" x="0" y="-1.27" size="1.778" layer="27" display="off"/>
+<attribute name="DESIGNER" value="Ian Lee" x="0" y="-1.27" size="1.778" layer="27" display="off"/>
+</element>
 </elements>
 <signals>
