File: Hardware/G2G-X Module/G2G-X Module.brd (EAGLE design)
At the start: 13.1 x 12.8 mm, 3 parts, among them J1 GROVE-4P-2.0-3470130P1

Commit message: Added frames to the U and X module schematics.
Parts:
- added FRAME1: (no value), SparkFun-Aesthetics:DUMMY
Changed lines of the file:
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@@
 <element name="LOGO1" library="SparkFun-Aesthetics" package="OSHW-LOGO-S" value="OSHW-LOGOS" x="1.8796" y="1.778" rot="MR0"/>
 <element name="U$1" library="SoftDust" package="2X5_1.27MM_FEMALE_PLUG" value="2X5_1.27MM_FEMALE_PLUG" x="6.5532" y="9.9822" rot="MR0"/>
+<element name="FRAME1" library="SparkFun-Aesthetics" package="DUMMY" value="" x="0" y="-1.27">
+<attribute name="VERSION" value="v1.0" x="0" y="-1.27" size="1.778" layer="27" display="off"/>
+<attribute name="DESIGNER" value="Ian Lee" x="0" y="-1.27" size="1.778" layer="27" display="off"/>
+</element>
 </elements>
 <signals>

Commit message: Added G2G-A and G2G-I modules.
Other:
- board text added: "Gadgeteer.in'"
- board text removed: "http://gadgeteer.in"
Changed lines of the file:
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@@
 <wire x1="12.2682" y1="9.9822" x2="12.2682" y2="11.8872" width="0.254" layer="21"/>
 <wire x1="12.2682" y1="11.8872" x2="10.3632" y2="11.8872" width="0.254" layer="21"/>
-<text x="9.7536" y="5.969" size="1.4224" layer="22" rot="MR0">G2G-X</text>
+<text x="12.5222" y="1.905" size="1.016" layer="22" rot="MR0">G2G-X</text>
 <text x="12.5222" y="0.6096" size="1.016" layer="22" rot="MR0">v1.0</text>
 <text x="2.6924" y="0.5588" size="0.8128" layer="21">D0</text>
@@
 <text x="6.7818" y="0.508" size="0.8128" layer="21">5V</text>
 <text x="9.0424" y="0.508" size="0.8128" layer="21">G</text>
-<text x="12.3952" y="2.8956" size="0.8128" layer="22" rot="MR0">http://gadgeteer.in</text>
+<text x="12.6238" y="5.7658" size="1.4224" layer="22" rot="MR0">Gadgeteer.in'</text>
 <rectangle x1="0.7225" y1="8.4731" x2="4.3801" y2="8.5493" layer="21"/>
 <rectangle x1="0.7225" y1="8.5493" x2="4.3801" y2="8.6255" layer="21"/>
