File: Hardware/G2G-I Module/G2G-I Module.sch (EAGLE design)
At the start: 4 parts, among them J1 GROVE-4P-2.0-3470130P1

Commit message: Replaced all 'G' logos with a new part for the logo.
Parts:
- added U$2: GADGETEER_LOGO_SMALL, SoftDust:GADGETEER_LOGO_SMALL
Changed lines of the file:
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@@
 <attribute name="VERSION" value="v1.0"/>
 </part>
+<part name="U$2" library="SoftDust" deviceset="GADGETEER_LOGO_SMALL" device=""/>
 </parts>
 <sheets>
@@
 <instance part="FRAME1" gate="G$1" x="0" y="0"/>
 <instance part="FRAME1" gate="V" x="147.32" y="0"/>
+<instance part="U$2" gate="G$1" x="40.64" y="10.16"/>
 </instances>
 <busses>
